File: RadioMusicHardware/RadioMusic.sch (EAGLE design)
At the start: 62 parts, among them IC2 7805L, IC3 TL072P, IC4 TL072P

Commit message: Renumber Parts
Parts:
- removed CHANNEL, TIME: 50k, TomW:ALPHA-9MMF2A
- removed CHANNEL_CV, OUT1, RESET, TIME_CV: WQP-PJ301M-12_JACK, thonkiconn:WQP-PJ301M-12_JACK
- removed IC4: TL072P, TomW:TL072P
- removed JP1BACK, JP1FRONT: M11LOCK, SparkFun-Connectors:M11LOCK
- removed RESET_BUTTON: D6_PUSH_SWITCH, TomW:D6_PUSH_SWITCH
- removed RESET_LED: (no value), TomW:LED3MM
- removed U$3: VERT_SD_CARD, TomW:VERT_SD_CARD
- removed VOLUME: (no value), bourns:3362P
- added IC1: TL072P, TomW:TL072P
- added J1, J2, J3, J4: WQP-PJ301M-12_JACK, thonkiconn:WQP-PJ301M-12_JACK
- added JP1, JP2: M11LOCK, SparkFun-Connectors:M11LOCK
- added LED5: (no value), TomW:LED3MM
- added R15: 1k, TomW:R-EU_STANDARD_RESISTOR
- added R22: 50k, TomW:ALPHA-9MMF2A
- added R8: 10k, TomW:R-EU_STANDARD_RESISTOR
- added S1: D6_PUSH_SWITCH, TomW:D6_PUSH_SWITCH
- added X1: VERT_SD_CARD, TomW:VERT_SD_CARD
- C1: value 10uf -> 1n; device SparkFun-Passives:CAP_POLPTH2 -> TomW:C-EU050-024X044
- C2: value 10uf -> 100n; device SparkFun-Passives:CAP_POLPTH2 -> TomW:C-EU050-025X075
- C3: value 1n -> 100n; device TomW:C-EU050-024X044 -> TomW:C-EU050-025X075
- C4: value 100n -> 1n
- C6: value 1n -> 10uf; device TomW:C-EU050-024X044 -> SparkFun-Passives:CAP_POLPTH2
- C7: value 100n -> 10uf; device TomW:C-EU050-025X075 -> SparkFun-Passives:CAP_POLPTH2
- C8: device TomW:C-EU050-025X075 -> TomW:C-EU050-024X044
- IC2: value 7805L -> TL072P; device gm-regulators:7805L -> TomW:TL072P
- IC3: value TL072P -> 7805L; device TomW:TL072P -> gm-regulators:7805L
- R1: value 100k -> 47R
- R10: value 100k -> 200k
- R11: value 200k -> 1k
- R12: value 47R -> 1k
- R13: value 100k -> 1k
- R14: value 220R -> 1k
- R16: value 10k -> 50k; device TomW:R-EU_STANDARD_RESISTOR -> TomW:ALPHA-9MMF2A
- R17, R18: value 1k -> 220R
- R19, R20: value 1k -> 100k
- R2: value 200k -> 47R
- R21: value 1k -> 200k
- R4: value 220R -> 8.2k
- R5: value 8.2k -> 330K
- R6: value 330K -> (none); device TomW:R-EU_STANDARD_RESISTOR -> bourns:3362P
- R9: value 47R -> 100k
- renumbered 1 to F1, FUSE to F2, JP2BACK to JP3, JP2FRONT to JP4, U$1 to U1
Connections:
- removed net N$12: IC3B.+IN, R10.2
- removed net N$8: IC4A.OUT, R4.2, VOLUME.2, VOLUME.3
- new net N$9: J1.2, R10.1, R9.1
- new net TEMP: J4.2, R20.1, R21.1
- net +12V: now also C5.1, C6.+, IC1P.V+, IC2P.V+, IC3.VI; no longer C1.+, C4.1, IC2.VI, IC3P.V+, IC4P.V+
- net +3.3V_F: now also R16.E, R22.E, S1.P, X1.VCC; no longer CHANNEL.E, RESET_BUTTON.P, TIME.E, U$3.VCC
- net +5V: now also IC3.VO; no longer IC2.VO
- net -12V: now also C7.-, C8.1, IC1P.V-, IC2P.V-; no longer C2.-, C5.1, IC3P.V-, IC4P.V-
- net AUDIO_OUT: now also IC2A.OUT, R6.2, R6.3; no longer R4.1
- net AUDIO_OUT_F: now also R17.2; no longer OUT1.2
- net CHANNEL_CV: now also IC1A.+IN; no longer R1.1, R2.1
- net CHANNEL_CV_F: now also R9.2; no longer CHANNEL_CV.2
- net CHANNEL_POT_F: now also R16.S; no longer CHANNEL.S
- net DAC: now also C2.1; no longer C8.1
- net DGND: now also C8.2, IC3.GND; no longer C4.2, IC2.GND
- net GND: now also C4.2, C6.-, C7.+, JP1.11, R10.2, R21.2, R5.1; no longer C1.-, C2.+, C6.2, JP1BACK.11, R11.2, R2.2, R6.1
- net GND_F: now also J1.1, J2.1, J3.1, J4.1, JP2.11, R11.1, R12.1, R14.2, R15.2, R16.A, R22.A, R8.2, X1.GND, X1.SHIELD@1, X1.SHIELD@2; no longer CHANNEL.A, CHANNEL_CV.1, JP1FRONT.11, OUT1.1, R16.2, R17.1, R18.1, R20.2, R21.2, RESET.1, TIME.A, TIME_CV.1, U$3.GND, U$3.SHIELD@1, U$3.SHIELD@2
- net LED1: now also JP1.1; no longer JP1BACK.1
- net LED1_F: now also JP2.1; no longer JP1FRONT.1
- net LED2: now also JP1.2; no longer JP1BACK.2
- net LED2_F: now also JP2.2; no longer JP1FRONT.2
- net LED3: now also JP1.3; no longer JP1BACK.3
- net LED3_F: now also JP2.3; no longer JP1FRONT.3
- net LED4: now also JP1.4; no longer JP1BACK.4
- net LED4_F: now also JP2.4; no longer JP1FRONT.4
- net LED_RESET: now also JP1.9; no longer JP1BACK.9
- net LED_RESET_F: now also JP2.9, LED5.A; no longer JP1FRONT.9, RESET_LED.A
- net MISO: now also JP1.10; no longer JP1BACK.10
- net MISO_F: now also JP2.10, X1.DO; no longer JP1FRONT.10, U$3.DO
- net MOSI: now also JP1.5; no longer JP1BACK.5
- net MOSI_F: now also JP2.5, X1.DI; no longer JP1FRONT.5, U$3.DI
- net N$1: now also IC1B.-IN, IC1B.OUT, R2.1; no longer IC3B.-IN, IC3B.OUT, R12.1
- net N$10: now also C2.2, R3.1; no longer C8.2, R5.1
- net N$14: now also J3.2, R18.1; no longer R14.1, RESET.2
- net N$18: now also R11.2; no longer R17.2
- net N$19: now also R12.2; no longer R18.2
- net N$2: now also C4.1, IC2B.+IN, R4.1; no longer C6.1, IC4B.+IN, R3.1
- net N$20: now also R13.2; no longer R19.2
- net N$21: now also R14.1; no longer R20.1
- net N$25: now also LED5.C, R15.1; no longer R21.1, RESET_LED.C
- net N$3: now also J2.2, R17.1; no longer IC3A.+IN, R1.2
- net N$4: now also C1.1, R4.2; no longer C3.1, R5.2
- net N$5: now also C1.2, IC2B.-IN, IC2B.OUT; no longer C7.2, IC4B.-IN, IC4B.OUT
- net N$6: now also C3.1, IC2A.+IN, R5.2; no longer C7.1, IC4A.+IN, R6.2
- net N$7: now also IC2A.-IN, R6.1; no longer IC4A.-IN, VOLUME.1
- net PIN20/A6: now also R2.2; no longer R12.2
- net PIN22/A8: now also IC1A.-IN, IC1A.OUT, R1.1, R1.2; no longer IC3A.-IN, IC3A.OUT, R9.1, R9.2
- net RESET_CV: now also JP1.7; no longer JP1BACK.7
- net RESET_CV_F: now also JP2.7, R18.2, R19.2; no longer JP1FRONT.7, R13.2, R14.2
- net RESET_SW: now also JP1.6; no longer JP1BACK.6
- net RESET_SW_F: now also JP2.6, R8.1, S1.O; no longer JP1FRONT.6, R16.1, RESET_BUTTON.O
- net SCLK_F: now also X1.SCK; no longer U$3.SCK
- net SS: now also JP1.8; no longer JP1BACK.8
- net SS_F: now also JP2.8, X1.CS; no longer JP1FRONT.8, U$3.CS
- net TIME_CV: now also IC1B.+IN; no longer R10.1, R11.1
- net TIME_CV_F: now also R20.2; no longer TIME_CV.2
- net TIME_POT_F: now also R22.S; no longer TIME.S
Other:
- note removed: "TEST: Should I take AGND to the front panel?"
- moved on the sheet: C3, C4, C5, C8, D7, D8, LED1, LED2, LED3, LED4, R1, R10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
