File: RadioMusicHardware/RadioMusic_Panel.sch (EAGLE design)
At the start: 13 parts, among them X1 VERT_SD_CARD

Commit message: Panel design
Parts:
- removed CHANNEL-CV, OUTPUT, RESET-CV, TIME-CV: WQP-PJ301M-12_JACK, thonkiconn:WQP-PJ301M-12_JACK
- removed CHANNEL-POT, TIME-POT: 50k, TomW:ALPHA-9MMF2A
- removed LED1, LED2, LED3, LED4, LED5: (no value), TomW:LED3MM
- removed RESET: D6_PUSH_SWITCH, TomW:D6_PUSH_SWITCH
- removed X1: VERT_SD_CARD, TomW:VERT_SD_CARD
Connections:
- removed net +3.3V_F: TIME-POT.E
- removed net GND_F: CHANNEL-CV.1
- removed net LED3_F: LED3.A
- removed net LED4_F: LED4.A
Other:
- note removed: "PJS008U-3000-0 microSD card holder"
- note removed: "ie D6R60 F1 LFS (Black, Round)"
Changed lines of the file:
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@@
 </classes>
 <parts>
-<part name="CHANNEL-POT" library="TomW" deviceset="ALPHA-9MM" device="A" technology="F2" value="50k"/>
-<part name="CHANNEL-CV" library="thonkiconn" deviceset="WQP-PJ301M-12_JACK" device="" value=""/>
-<part name="RESET-CV" library="thonkiconn" deviceset="WQP-PJ301M-12_JACK" device="" value=""/>
-<part name="OUTPUT" library="thonkiconn" deviceset="WQP-PJ301M-12_JACK" device="" value=""/>
-<part name="TIME-POT" library="TomW" deviceset="ALPHA-9MM" device="A" technology="F2" value="50k"/>
-<part name="TIME-CV" library="thonkiconn" deviceset="WQP-PJ301M-12_JACK" device="" value=""/>
-<part name="RESET" library="TomW" deviceset="D6_PUSH_SWITCH" device="" value="D6_PUSH_SWITCH"/>
-<part name="LED1" library="TomW" deviceset="LED" device="3MM"/>
-<part name="LED2" library="TomW" deviceset="LED" device="3MM"/>
-<part name="LED3" library="TomW" deviceset="LED" device="3MM"/>
-<part name="LED4" library="TomW" deviceset="LED" device="3MM"/>
-<part name="X1" library="TomW" deviceset="VERT_SD_CARD" device=""/>
-<part name="LED5" library="TomW" deviceset="LED" device="3MM"/>
 </parts>
 <sheets>
 <sheet>
 <plain>
-<text x="83.82" y="144.78" size="1.778" layer="91">ie D6R60 F1 LFS (Black, Round)</text>
-<text x="152.4" y="142.24" size="1.778" layer="91">PJS008U-3000-0 microSD card holder</text>
-<text x="152.4" y="142.24" size="1.778" layer="91">PJS008U-3000-0 microSD card holder</text>
 </plain>
 <instances>
-<instance part="CHANNEL-POT" gate="G$1" x="25.4" y="81.28"/>
-<instance part="CHANNEL-CV" gate="G$1" x="30.48" y="114.3" rot="MR0"/>
-<instance part="RESET-CV" gate="G$1" x="81.28" y="40.64" rot="MR0"/>
-<instance part="OUTPUT" gate="G$1" x="149.86" y="71.12"/>
-<instance part="TIME-POT" gate="G$1" x="30.48" y="22.86"/>
-<instance part="TIME-CV" gate="G$1" x="30.48" y="53.34" rot="MR0"/>
-<instance part="RESET" gate="G$1" x="99.06" y="137.16"/>
-<instance part="LED1" gate="G$1" x="157.48" y="45.72" rot="R270"/>
-<instance part="LED2" gate="G$1" x="157.48" y="38.1" rot="R270"/>
-<instance part="LED3" gate="G$1" x="157.48" y="30.48" rot="R270"/>
-<instance part="LED4" gate="G$1" x="157.48" y="22.86" rot="R270"/>
-<instance part="X1" gate="G$1" x="162.56" y="121.92"/>
-<instance part="LED5" gate="G$1" x="157.48" y="15.24" rot="R270"/>
 </instances>
 <busses>
 </busses>
 <nets>
-<net name="LED4_F" class="0">
-<segment>
-<pinref part="LED4" gate="G$1" pin="A"/>
-<wire x1="162.56" y1="22.86" x2="160.02" y2="22.86" width="0.1524" layer="91"/>
-</segment>
-</net>
-<net name="LED3_F" class="0">
-<segment>
-<pinref part="LED3" gate="G$1" pin="A"/>
-<wire x1="162.56" y1="30.48" x2="160.02" y2="30.48" width="0.1524" layer="91"/>
-</segment>
-</net>
-<net name="+3.3V_F" class="0">
-<segment>
-<pinref part="TIME-POT" gate="G$1" pin="E"/>
-<wire x1="30.48" y1="33.02" x2="30.48" y2="30.48" width="0.1524" layer="91"/>
-</segment>
-</net>
-<net name="GND_F" class="2">
-<segment>
-<pinref part="CHANNEL-CV" gate="G$1" pin="1"/>
-<wire x1="35.56" y1="109.22" x2="35.56" y2="111.76" width="0.1524" layer="91"/>
-<label x="35.56" y="109.22" size="1.016" layer="95" rot="R270" xref="yes"/>
-</segment>
-</net>
 </nets>
 </sheet>
