File: RadioMusicHardware/RadioMusic_B.sch (EAGLE design)
At the start: 32 parts, among them IC1 TL072P, IC2 TL072P, IC3 7805L, U1 TEENSY_3.1_TW

Commit message: Back board reworking
Parts:
- removed IC1, IC2: TL072P, TomW:TL072P
- added IC4: TL074, linear:TL074P
- JP1: value M11LOCK -> M11PTH; device SparkFun-Connectors:M11LOCK -> SparkFun-Connectors:M11PTH
- JP3: device SparkFun-Connectors:M07LOCK -> SparkFun-Connectors:M07
- renumbered R6 to OUTPUT
Connections:
- new net N$3: IC4B.-IN, IC4B.OUT, R1.2
- net +12V: now also C5.2, IC4P.V+; no longer C5.1, IC1P.V+, IC2P.V+
- net -12V: now also C8.2, IC4P.V-; no longer C8.1, IC1P.V-, IC2P.V-
- net AUDIO_OUT: now also IC4A.OUT; no longer IC2A.OUT
- net CHANNEL_CV: now also IC4B.+IN; no longer IC1A.+IN
- net DGND: no longer C5.2, C8.2
- net GND: now also C5.1, C8.1, JP1.1, R7.2; no longer JP1.11, R7.1
- net LED1: now also JP1.2; no longer JP1.1
- net LED2: now also JP1.3; no longer JP1.2
- net LED3: now also JP1.4; no longer JP1.3
- net LED4: now also JP1.5; no longer JP1.4
- net LED_RESET: now also JP1.10; no longer JP1.9
- net MISO: now also JP1.11; no longer JP1.10
- net MOSI: now also JP1.6; no longer JP1.5
- net N$1: now also IC4C.-IN, IC4C.OUT, R2.2; no longer IC1B.-IN, IC1B.OUT, R2.1
- net N$10: now also R3.2; no longer R3.1
- net N$2: now also IC4D.+IN, R4.2; no longer IC2B.+IN, R4.1
- net N$4: now also R3.1, R4.1; no longer R3.2, R4.2
- net N$5: now also C3.1, IC4D.-IN, IC4D.OUT; no longer C3.2, IC2B.-IN, IC2B.OUT
- net N$6: now also C3.2, IC4A.+IN; no longer C3.1, IC2A.+IN
- net N$7: now also IC4A.-IN, R7.1; no longer IC2A.-IN, R7.2
- net PIN20/A6: now also R2.1; no longer R2.2
- net PIN22/A8: no longer IC1A.-IN, IC1A.OUT, R1.2
- net RESET_CV: now also JP1.8; no longer JP1.7
- net RESET_SW: now also JP1.7; no longer JP1.6
- net SS: now also JP1.9; no longer JP1.8
- net TIME_CV: now also IC4C.+IN; no longer IC1B.+IN
Other:
- moved on the sheet: C5, JP1, R1, R2, R3, R4

Commit message: PCB cosmetic changes
Other:
- moved on the sheet: C1, C2, C3, R7
Changed lines of the file:
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@@
 <part name="U1" library="TomW" deviceset="TEENSY_3.1_TW" device=""/>
 <part name="IC3" library="gm-regulators" deviceset="78*" device="L" technology="05"/>
-<part name="D1" library="diode" deviceset="BAT81" device="" value=""/>
-<part name="D2" library="diode" deviceset="BAT81" device="" value=""/>
+<part name="D1" library="diode" deviceset="BAT81" device="" value="BAT81"/>
+<part name="D2" library="diode" deviceset="BAT81" device="" value="BAT81"/>
 <part name="R4" library="TomW" deviceset="R-EU_" device="STANDARD_RESISTOR" value="8.2k"/>
 <part name="R3" library="TomW" deviceset="R-EU_" device="STANDARD_RESISTOR" value="8.2k"/>
@@
 <part name="C2" library="TomW" deviceset="C-EU" device="050-025X075" value="100n"/>
 <part name="R1" library="TomW" deviceset="R-EU_" device="STANDARD_RESISTOR" value="47R"/>
-<part name="D3" library="diode" deviceset="BAT81" device="" value=""/>
-<part name="D4" library="diode" deviceset="BAT81" device="" value=""/>
+<part name="D3" library="diode" deviceset="BAT81" device="" value="BAT81"/>
+<part name="D4" library="diode" deviceset="BAT81" device="" value="BAT81"/>
 <part name="R2" library="TomW" deviceset="R-EU_" device="STANDARD_RESISTOR" value="47R"/>
 <part name="L1" library="inductors" deviceset="BL0" device="1RN1A"/>
@@
 <instance part="R4" gate="G$1" x="162.56" y="73.66"/>
 <instance part="R3" gate="G$1" x="142.24" y="73.66" rot="R180"/>
-<instance part="C1" gate="G$1" x="175.26" y="83.82" rot="R270"/>
+<instance part="C1" gate="G$1" x="175.26" y="83.82" rot="R90"/>
 <instance part="C4" gate="G$1" x="170.18" y="58.42"/>
-<instance part="C3" gate="G$1" x="205.74" y="71.12" rot="R270"/>
+<instance part="C3" gate="G$1" x="205.74" y="71.12" rot="R90"/>
 <instance part="R5" gate="G$1" x="213.36" y="58.42" rot="R90"/>
-<instance part="R7" gate="G$1" x="220.98" y="48.26" rot="R90"/>
-<instance part="C2" gate="G$1" x="129.54" y="73.66" rot="R270"/>
+<instance part="R7" gate="G$1" x="220.98" y="48.26" rot="R270"/>
+<instance part="C2" gate="G$1" x="129.54" y="73.66" rot="R90"/>
 <instance part="R1" gate="G$1" x="35.56" y="114.3" rot="R180"/>
 <instance part="IC4" gate="C" x="17.78" y="60.96"/>
@@
 <segment>
 <pinref part="R7" gate="G$1" pin="2"/>
-<wire x1="220.98" y1="40.64" x2="220.98" y2="53.34" width="0.1524" layer="91"/>
+<wire x1="220.98" y1="40.64" x2="220.98" y2="43.18" width="0.1524" layer="91"/>
 <pinref part="R5" gate="G$1" pin="1"/>
 <wire x1="213.36" y1="40.64" x2="213.36" y2="53.34" width="0.1524" layer="91"/>
@@
 <segment>
 <pinref part="C2" gate="G$1" pin="1"/>
-<wire x1="119.38" y1="73.66" x2="132.08" y2="73.66" width="0.1524" layer="91"/>
+<wire x1="119.38" y1="73.66" x2="127" y2="73.66" width="0.1524" layer="91"/>
 <label x="119.38" y="73.66" size="1.778" layer="95" rot="R180" xref="yes"/>
 </segment>
@@
 <pinref part="C1" gate="G$1" pin="1"/>
 <wire x1="152.4" y1="73.66" x2="157.48" y2="73.66" width="0.1524" layer="91"/>
-<wire x1="177.8" y1="83.82" x2="152.4" y2="83.82" width="0.1524" layer="91"/>
+<wire x1="172.72" y1="83.82" x2="152.4" y2="83.82" width="0.1524" layer="91"/>
 <wire x1="152.4" y1="83.82" x2="152.4" y2="73.66" width="0.1524" layer="91"/>
 <junction x="152.4" y="73.66"/>
@@
 <segment>
 <pinref part="C1" gate="G$1" pin="2"/>
-<wire x1="170.18" y1="83.82" x2="195.58" y2="83.82" width="0.1524" layer="91"/>
+<wire x1="180.34" y1="83.82" x2="195.58" y2="83.82" width="0.1524" layer="91"/>
 <wire x1="195.58" y1="83.82" x2="195.58" y2="71.12" width="0.1524" layer="91"/>
 <pinref part="IC4" gate="D" pin="OUT"/>
@@
 <junction x="195.58" y="71.12"/>
 <pinref part="C3" gate="G$1" pin="1"/>
-<wire x1="208.28" y1="71.12" x2="195.58" y2="71.12" width="0.1524" layer="91"/>
+<wire x1="203.2" y1="71.12" x2="195.58" y2="71.12" width="0.1524" layer="91"/>
 </segment>
 </net>
@@
 <pinref part="C3" gate="G$1" pin="2"/>
 <pinref part="IC4" gate="A" pin="+IN"/>
-<wire x1="200.66" y1="71.12" x2="213.36" y2="71.12" width="0.1524" layer="91"/>
+<wire x1="210.82" y1="71.12" x2="213.36" y2="71.12" width="0.1524" layer="91"/>
 <wire x1="213.36" y1="71.12" x2="223.52" y2="71.12" width="0.1524" layer="91"/>
 <wire x1="213.36" y1="71.12" x2="213.36" y2="63.5" width="0.1524" layer="91"/>
@@
 <wire x1="223.52" y1="66.04" x2="220.98" y2="66.04" width="0.1524" layer="91"/>
 <wire x1="220.98" y1="66.04" x2="220.98" y2="58.42" width="0.1524" layer="91"/>
-<wire x1="220.98" y1="58.42" x2="220.98" y2="43.18" width="0.1524" layer="91"/>
+<wire x1="220.98" y1="58.42" x2="220.98" y2="53.34" width="0.1524" layer="91"/>
 <wire x1="226.06" y1="58.42" x2="220.98" y2="58.42" width="0.1524" layer="91"/>
 <junction x="220.98" y="58.42"/>
@@
 <pinref part="R3" gate="G$1" pin="2"/>
 <pinref part="C2" gate="G$1" pin="2"/>
-<wire x1="124.46" y1="73.66" x2="137.16" y2="73.66" width="0.1524" layer="91"/>
-</segment>
-</net>
+<wire x1="134.62" y1="73.66" x2="137.16" y2="73.66" width="0.1524" layer="91"/>
+</segment>
+</net>
