File: RadioMusicHardware/RadioMusic_F.brd (EAGLE design)
At the start: 107 x 19 mm, 31 parts, among them X1 VERT_SD_CARD

Commit message: Text subbing
Parts:
- turned R14 to 0 degrees
Connections:
- net GND_F: now also R14.1; no longer R14.2
- net N$21: now also R14.2; no longer R14.1
Other:
- board text added: "-->"
- board text added: "<-BAT81 x2"
- board text added: "Be super careful with LED Polarity up here -->"
- board text added: "Header Pins THIS SIDE"
- board text added: "Radio Music Front PCB rev 1 Designed in Herne Hill, London by Tom Whitwell October 2014 CC-BY-SA musicthing.co.uk"
- board text removed: "ONLY JUMPER PINS ON THIS SIDE"
- board text removed: "RadioMusic Front PCB rev 1 Designed in Herne Hill, London by Tom Whitwell October 2014 CC-BY-SA musicthing.co.uk"
Changed lines of the file:
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@@
 <grid distance="25" unitdist="mil" unit="mil" style="lines" multiple="1" display="yes" altdistance="8" altunitdist="mil" altunit="mil"/>
 <layers>
-<layer number="1" name="Top" color="4" fill="1" visible="no" active="yes"/>
+<layer number="1" name="Top" color="4" fill="1" visible="yes" active="yes"/>
 <layer number="2" name="Route2" color="1" fill="3" visible="no" active="yes"/>
 <layer number="3" name="Route3" color="4" fill="3" visible="no" active="no"/>
 <layer number="14" name="Route14" color="1" fill="6" visible="no" active="no"/>
 <layer number="15" name="Route15" color="4" fill="6" visible="no" active="yes"/>
-<layer number="16" name="Bottom" color="1" fill="1" visible="no" active="yes"/>
+<layer number="16" name="Bottom" color="1" fill="1" visible="yes" active="yes"/>
 <layer number="17" name="Pads" color="2" fill="1" visible="yes" active="yes"/>
 <layer number="18" name="Vias" color="2" fill="1" visible="yes" active="yes"/>
 <layer number="19" name="Unrouted" color="6" fill="1" visible="no" active="yes"/>
 <layer number="20" name="Dimension" color="15" fill="1" visible="yes" active="yes"/>
-<layer number="21" name="tPlace" color="7" fill="1" visible="no" active="yes"/>
-<layer number="22" name="bPlace" color="7" fill="1" visible="yes" active="yes"/>
-<layer number="23" name="tOrigins" color="15" fill="1" visible="no" active="yes"/>
-<layer number="24" name="bOrigins" color="15" fill="1" visible="yes" active="yes"/>
-<layer number="25" name="tNames" color="7" fill="1" visible="no" active="yes"/>
+<layer number="21" name="tPlace" color="7" fill="1" visible="yes" active="yes"/>
+<layer number="22" name="bPlace" color="7" fill="1" visible="no" active="yes"/>
+<layer number="23" name="tOrigins" color="15" fill="1" visible="yes" active="yes"/>
+<layer number="24" name="bOrigins" color="15" fill="1" visible="no" active="yes"/>
+<layer number="25" name="tNames" color="7" fill="1" visible="yes" active="yes"/>
 <layer number="26" name="bNames" color="7" fill="1" visible="no" active="yes"/>
-<layer number="27" name="tValues" color="7" fill="1" visible="no" active="yes"/>
+<layer number="27" name="tValues" color="7" fill="1" visible="yes" active="yes"/>
 <layer number="28" name="bValues" color="7" fill="1" visible="no" active="yes"/>
 <layer number="29" name="tStop" color="7" fill="3" visible="no" active="yes"/>
@@
 <wire x1="120" y1="9.5" x2="-20" y2="9.5" width="0.1" layer="51"/>
 <wire x1="53.5" y1="-10" x2="53.5" y2="30" width="0.1" layer="51"/>
-<text x="25.4" y="5.715" size="1.016" layer="22" rot="MR0">RadioMusic Front PCB rev 1
+<text x="25.4" y="5.715" size="1.016" layer="22" rot="MR0">Radio Music Front PCB rev 1
 Designed in Herne Hill,
 London by Tom Whitwell
 October 2014 CC-BY-SA
 musicthing.co.uk</text>
-<text x="74.93" y="7.62" size="1.27" layer="22" rot="MR0">ONLY
-JUMPER PINS
-ON THIS SIDE </text>
+<text x="74.93" y="7.62" size="1.27" layer="22" rot="MR0">Header Pins
+THIS SIDE</text>
+<text x="70.485" y="11.43" size="1.27" layer="22" rot="MR90">--&gt;</text>
+<text x="71.755" y="6.985" size="1.27" layer="22" rot="SMR270">--&gt;</text>
+<text x="36.3474" y="13.9192" size="0.762" layer="21" rot="R90" align="center-left">&lt;-BAT81
+   x2</text>
+<text x="74.0664" y="0.7112" size="0.762" layer="21" distance="40">Be super careful with
+LED Polarity up here --&gt;</text>
 </plain>
 <attributes>
@@
 <attribute name="VALUE" x="90.83" y="11.485" size="0.6096" layer="27" rot="R270"/>
 </element>
-<element name="CHANNEL-CV" library="thonkiconn" package="WQP-PJ301M-12_JACK" value="" x="20.955" y="4.445" rot="R90"/>
-<element name="RESET-CV" library="thonkiconn" package="WQP-PJ301M-12_JACK" value="" x="6.35" y="14.605" rot="R90"/>
-<element name="OUTPUT" library="thonkiconn" package="WQP-PJ301M-12_JACK" value="" x="6.35" y="4.445" rot="R90"/>
+<element name="CHANNEL-CV" library="thonkiconn" package="WQP-PJ301M-12_JACK" value="" x="20.955" y="4.445" smashed="yes" rot="R90">
+<attribute name="NAME" x="24.6126" y="1.3208" size="1.016" layer="21" rot="R180"/>
+</element>
+<element name="RESET-CV" library="thonkiconn" package="WQP-PJ301M-12_JACK" value="" x="6.35" y="14.605" smashed="yes" rot="R90">
+<attribute name="NAME" x="8.1788" y="11.2776" size="1.016" layer="21" rot="R180"/>
+</element>
+<element name="OUTPUT" library="thonkiconn" package="WQP-PJ301M-12_JACK" value="" x="6.35" y="4.445" smashed="yes" rot="R90">
+<attribute name="NAME" x="6.35" y="1.3208" size="1.016" layer="21" rot="R180"/>
+</element>
 <element name="R9" library="TomW" package="0207/10" value="100k" x="57.785" y="9.525" rot="R90"/>
 <element name="R10" library="TomW" package="0207/10" value="200k" x="84.455" y="9.525" rot="R90"/>
@@
 <attribute name="VALUE" x="63.5" y="13.335" size="0.6096" layer="27" rot="R270"/>
 </element>
-<element name="TIME-CV" library="thonkiconn" package="WQP-PJ301M-12_JACK" value="" x="20.955" y="14.605" rot="R90"/>
+<element name="TIME-CV" library="thonkiconn" package="WQP-PJ301M-12_JACK" value="" x="20.955" y="14.605" smashed="yes" rot="R90">
+<attribute name="NAME" x="21.3614" y="11.2776" size="1.016" layer="21" rot="R180"/>
+</element>
 <element name="R20" library="TomW" package="0207/10" value="100k" x="76.835" y="9.525" rot="R90"/>
 <element name="R21" library="TomW" package="0207/10" value="200k" x="79.375" y="9.525" rot="R90"/>
-<element name="D7" library="diode" package="DO34-7" value="BAT81" x="36.83" y="9.525" rot="R90"/>
-<element name="D8" library="diode" package="DO34-7" value="BAT81" x="34.925" y="9.525" rot="R270"/>
+<element name="D7" library="diode" package="DO34-7" value="BAT81" x="36.83" y="9.525" smashed="yes" rot="R90"/>
+<element name="D8" library="diode" package="DO34-7" value="BAT81" x="34.925" y="9.525" smashed="yes" rot="R270"/>
 <element name="R19" library="TomW" package="0207/10" value="100k" x="32.385" y="9.525" rot="R90"/>
 <element name="R18" library="TomW" package="0207/10" value="220R" x="29.845" y="9.525" rot="R90"/>
-<element name="RESET" library="TomW" package="D6_BUTTON_RND" value="D6_PUSH_SWITCH" x="44.45" y="6.35" rot="R180"/>
+<element name="RESET" library="TomW" package="D6_BUTTON_RND" value="D6_PUSH_SWITCH" x="44.45" y="6.35" smashed="yes" rot="R180">
+<attribute name="NAME" x="49.1744" y="3.81" size="1.27" layer="25" rot="R90"/>
+</element>
 <element name="R8" library="TomW" package="0207/10" value="10k" x="32.385" y="1.905"/>
 <element name="LED1" library="TomW" package="LED3MM" value="" x="105.156" y="16.256" rot="R90"/>
@@
 <element name="R12" library="TomW" package="0207/10" value="1k" x="102.235" y="9.525" rot="R90"/>
 <element name="R13" library="TomW" package="0207/10" value="1k" x="81.915" y="9.525" rot="R90"/>
-<element name="R14" library="TomW" package="0207/10" value="1k" x="95.885" y="1.905" rot="R180"/>
+<element name="R14" library="TomW" package="0207/10" value="1k" x="95.885" y="1.905"/>
 <element name="X1" library="TomW" package="VERT_MICROSD" value="VERT_SD_CARD" x="44.45" y="16.51"/>
 <element name="LED5" library="TomW" package="LED3MM" value="" x="52.705" y="3.175" rot="R270"/>
@@
 <signal name="N$21">
 <contactref element="LED4" pad="K"/>
-<contactref element="R14" pad="1"/>
+<contactref element="R14" pad="2"/>
 <wire x1="105.0544" y1="1.8288" x2="100.9904" y2="1.8288" width="0.3048" layer="1"/>
 <wire x1="100.9904" y1="1.8288" x2="100.965" y2="1.905" width="0.3048" layer="1"/>
@@
 <contactref element="R12" pad="1"/>
 <contactref element="R13" pad="1"/>
-<contactref element="R14" pad="2"/>
+<contactref element="R14" pad="1"/>
 <contactref element="R15" pad="2"/>
 <contactref element="OUTPUT" pad="P$3"/>
