File: RadioMusicHardware/RadioMusic_F.sch (EAGLE design)
At the start: 30 parts, among them X1 VERT_SD_CARD_REV2

Commit message: Fix Button colour on Eagle Schematic
Other:
- note added: "ie D6R90 F1 LFS (Black, Round)"
- note removed: "ie D6R60 F1 LFS (Black, Round)"
Changed lines of the file:
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@@
 <sheet>
 <plain>
-<text x="83.82" y="144.78" size="1.778" layer="91">ie D6R60 F1 LFS (Black, Round)</text>
+<text x="83.82" y="144.78" size="1.778" layer="91">ie D6R90 F1 LFS (Black, Round)</text>
 <text x="152.4" y="142.24" size="1.778" layer="91">PJS008U-3000-0 microSD card holder</text>
 <text x="152.4" y="142.24" size="1.778" layer="91">PJS008U-3000-0 microSD card holder</text>
